File: pcb/bbk.kicad_sch (KiCad schematic)
At the start: 54 parts, among them J1 TagConnect, J2 USB_C_Receptacle_USB2.0, J3 Neopixel, J4 Conn_01x04, J5 Conn_01x03, J6 Conn_01x02, Q1 Q_NMOS_SGD, SW1 Reset, U1 AP7370-33W5-7, U2 MP2667GG-xxxx-Z, U3 STM32G0xxFx, U4 STSPIN240, U5 TSOP93338

Commit message: cleanup
Parts:
- C1: value C -> 10uF
- C10, C2, C5, C7: renamed from C1; value C -> 100nF
- C12: renamed from C1; value C -> 22nF
- C3, C4, C6, C8, C9: renamed from C1; value C -> 10uF
- FB1: footprint (none) -> Resistor_SMD:R_0603_1608Metric
- J2: renamed from J3; footprint (none) -> Connector_JST:JST_SH_BM03B-SRSS-TB_1x03-1MP_P1.00mm_Vertical
- J3: renamed from J6; value Conn_01x02 -> ExtPower; footprint (none) -> Connector_PinHeader_2.54mm:PinHeader_1x02_P2.54mm_Vertical
- J5: value Conn_01x03 -> Li-Ion; footprint (none) -> Connector_JST:JST_SH_BM03B-SRSS-TB_1x03-1MP_P1.00mm_Vertical
- J6: renamed from J4; value Conn_01x04 -> I2C; footprint (none) -> Connector_JST:JST_SH_BM04B-SRSS-TB_1x04-1MP_P1.00mm_Vertical
- J7: renamed from J4; value Conn_01x04 -> Motors; footprint (none) -> Connector_JST:JST_SH_BM04B-SRSS-TB_1x04-1MP_P1.00mm_Vertical
- Q1: value Q_NMOS_SGD -> PMV15ENEA
- R1: value R -> 10K; footprint (none) -> Resistor_SMD:R_0603_1608Metric
- R10, R2, R5: renamed from R1; value R -> 190R; footprint (none) -> Resistor_SMD:R_0603_1608Metric
- R11: renamed from R1; value R -> 330R; footprint (none) -> Resistor_SMD:R_0603_1608Metric
- R12, R20, R6, R7, R9: renamed from R1; value R -> 10K; footprint (none) -> Resistor_SMD:R_0603_1608Metric
- R13, R18, R19, R3, R4: renamed from R1; value R -> 5.1K; footprint (none) -> Resistor_SMD:R_0603_1608Metric
- R14: renamed from R1; value R -> 47K; footprint (none) -> Resistor_SMD:R_0603_1608Metric
- R15: renamed from R1; value R -> 1K; footprint (none) -> Resistor_SMD:R_0603_1608Metric
- R16, R17: renamed from R1; value R -> 2R; footprint (none) -> Resistor_SMD:R_0603_1608Metric
- R8: renamed from R1; value R -> 20K; footprint (none) -> Resistor_SMD:R_0603_1608Metric
- SW1: footprint Resistor_SMD:R_1210_3225Metric -> Resistor_SMD:R_1206_3216Metric_Pad1.30x1.75mm_HandSolder
- SW2: renamed from SW1; value Reset -> Wakeup; footprint Resistor_SMD:R_1210_3225Metric -> Resistor_SMD:R_1206_3216Metric_Pad1.30x1.75mm_HandSolder
- U4: renamed from U1; footprint Package_TO_SOT_SMD:TSOT-23-5_HandSoldering -> Package_TO_SOT_SMD:TSOT-23-5
- renumbered C9 to C11, H1 to H2, H1 to H3, H1 to H4, J2 to J1, J1 to J4, U3 to U1, U5 to U3, U4 to U5
